File: STM32/lc_meter.sch (EAGLE design)
At the start: 40 parts, among them IC1 LM311N, IC2 REG1117, IC3 REG1117, K1 REED, K2 REED, Q1 16MHz, T1 2n2222, T2 2n2222, U1 STM32F030XTSSOP20

Commit message: Add files via upload
Connections:
- removed net N$4: INDUCTANCE.1, K12.S, U$1.1
- new net N$26: INDUCTANCE.2, K12.S, U$1.1
- net GND: now also INDUCTANCE.1
- net N$3: no longer INDUCTANCE.2
Other:
- moved on the sheet: INDUCTANCE
Changed lines of the file:
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@@
 <attribute name="VALUE" x="48.26" y="121.92" size="1.778" layer="96" rot="R90"/>
 </instance>
-<instance part="INDUCTANCE" gate="G$1" x="-129.54" y="78.74" smashed="yes" rot="R180">
-<attribute name="NAME" x="-130.81" y="83.185" size="1.778" layer="95"/>
-<attribute name="VALUE" x="-123.19" y="83.82" size="1.778" layer="96" rot="R180"/>
+<instance part="INDUCTANCE" gate="G$1" x="-129.54" y="43.18" smashed="yes" rot="R180">
+<attribute name="NAME" x="-130.81" y="47.625" size="1.778" layer="95"/>
+<attribute name="VALUE" x="-123.19" y="48.26" size="1.778" layer="96" rot="R180"/>
 </instance>
 </instances>
@@
 <wire x1="-58.42" y1="40.64" x2="-68.58" y2="40.64" width="0.1524" layer="91"/>
 <junction x="-68.58" y="40.64"/>
+<pinref part="INDUCTANCE" gate="G$1" pin="1"/>
+<wire x1="-127" y1="40.64" x2="-111.76" y2="40.64" width="0.1524" layer="91"/>
 </segment>
 <segment>
@@
 <wire x1="-99.06" y1="78.74" x2="-83.82" y2="78.74" width="0.1524" layer="91"/>
 <wire x1="-83.82" y1="78.74" x2="-78.74" y2="78.74" width="0.1524" layer="91"/>
-<wire x1="-127" y1="78.74" x2="-111.76" y2="78.74" width="0.1524" layer="91"/>
-<junction x="-111.76" y="78.74"/>
 <pinref part="C1" gate="G$1" pin="2"/>
 <pinref part="C3-CAL" gate="G$1" pin="1"/>
@@
 <wire x1="-83.82" y1="68.58" x2="-83.82" y2="78.74" width="0.1524" layer="91"/>
 <junction x="-83.82" y="78.74"/>
-<pinref part="INDUCTANCE" gate="G$1" pin="2"/>
-</segment>
-</net>
-<net name="N$4" class="0">
-<segment>
-<pinref part="U$1" gate="L$1" pin="1"/>
-<pinref part="K1" gate="2" pin="S"/>
-<wire x1="-111.76" y1="50.8" x2="-111.76" y2="53.34" width="0.1524" layer="91"/>
-<wire x1="-111.76" y1="53.34" x2="-111.76" y2="55.88" width="0.1524" layer="91"/>
-<wire x1="-111.76" y1="53.34" x2="-119.38" y2="53.34" width="0.1524" layer="91"/>
-<wire x1="-119.38" y1="53.34" x2="-119.38" y2="76.2" width="0.1524" layer="91"/>
-<junction x="-111.76" y="53.34"/>
-<wire x1="-119.38" y1="76.2" x2="-127" y2="76.2" width="0.1524" layer="91"/>
-<pinref part="INDUCTANCE" gate="G$1" pin="1"/>
 </segment>
 </net>
@@
 </segment>
 </net>
+<net name="N$26" class="0">
+<segment>
+<pinref part="U$1" gate="L$1" pin="1"/>
+<pinref part="K1" gate="2" pin="S"/>
+<wire x1="-111.76" y1="50.8" x2="-111.76" y2="53.34" width="0.1524" layer="91"/>
+<pinref part="INDUCTANCE" gate="G$1" pin="2"/>
+<wire x1="-111.76" y1="53.34" x2="-111.76" y2="55.88" width="0.1524" layer="91"/>
+<wire x1="-127" y1="43.18" x2="-119.38" y2="43.18" width="0.1524" layer="91"/>
+<wire x1="-119.38" y1="43.18" x2="-119.38" y2="53.34" width="0.1524" layer="91"/>
+<wire x1="-119.38" y1="53.34" x2="-111.76" y2="53.34" width="0.1524" layer="91"/>
+<junction x="-111.76" y="53.34"/>
+</segment>
+</net>
